File: PhantomBoard/PhantomBoard.sch (KiCad schematic (older format))
At the start: 26 parts, among them J1 XLR3, J2 AudioJack2, J3 XLR3, SW1 SW_SPDT, SW2 SW_SPDT, U1 XL6009

Commit message: schematic fixed
Connections:
- net at U1.5 (FB): now also R7.2, SW1.2 (B)
Changed lines of the file:
@@
 	1    0    0    -1
 $EndComp
+Wire Wire Line
+	6250 4350 7050 4350
+Wire Wire Line
+	6250 4250 6250 4350
+Connection ~ 7050 4350
 $EndSCHEMATC
